Commit message: feat: configure native CPU and GPU world-frame lidar scans

File: xgc2_simple_lidar/models/sensor.sdf.xacro (robot description, xacro)
@@ -9,6 +9,8 @@
   <xacro:arg name="layers" default="16"/>
   <xacro:arg name="vertical_fov" default="1.0"/>
+  <xacro:arg name="horizontal_fov" default="6.283185307179586"/>
+  <xacro:arg name="acceleration" default="gpu"/>
   <xacro:xgc2_simple_lidar_sensor namespace="$(arg namespace)" pose="$(arg pose)"
     rate="$(arg rate)" max_range="$(arg max_range)" samples="$(arg samples)"
-    layers="$(arg layers)" vertical_fov="$(arg vertical_fov)"/>
+    layers="$(arg layers)" vertical_fov="$(arg vertical_fov)" horizontal_fov="$(arg horizontal_fov)" acceleration="$(arg acceleration)"/>
 </sdf>

File: xgc2_simple_lidar/models/sensor.xacro (robot description, xacro)
@@ -1,6 +1,6 @@
 <?xml version="1.0"?>
 <robot xmlns:xacro="http://www.ros.org/wiki/xacro">
-  <xacro:macro name="xgc2_simple_lidar_sensor" params="namespace pose rate:=10 max_range:=20 samples:=360 layers:=16 vertical_fov:=1.0">
-    <sensor name="simple_lidar" type="gpu_ray">
+  <xacro:macro name="xgc2_simple_lidar_sensor" params="namespace pose rate:=10 max_range:=20 samples:=360 layers:=16 vertical_fov:=1.0 horizontal_fov:=${2*pi} acceleration:=gpu">
+    <sensor name="simple_lidar" type="${dict(cpu='ray', gpu='gpu_ray')[acceleration]}">
       <pose>${pose}</pose>
       <always_on>false</always_on>
@@ -11,5 +11,5 @@
           <horizontal>
             <samples>${samples}</samples><resolution>1</resolution>
-            <min_angle>-${pi}</min_angle><max_angle>${pi}</max_angle>
+            <min_angle>${-horizontal_fov / 2}</min_angle><max_angle>${horizontal_fov / 2}</max_angle>
           </horizontal>
           <vertical>
@@ -20,5 +20,5 @@
         <range><min>0.15</min><max>${max_range}</max><resolution>0.01</resolution></range>
       </ray>
-      <plugin name="simple_lidar" filename="libxgc2_simple_lidar.so">
+      <plugin name="simple_lidar" filename="${dict(cpu='libxgc2_simple_lidar_cpu.so', gpu='libxgc2_simple_lidar.so')[acceleration]}">
         <robotNamespace>${namespace}</robotNamespace>
       </plugin>

Commit message: Define the simple lidar scan defaults once.
The macro parameters in sensor.xacro and the arguments of the
sensor.sdf.xacro wrapper each restated rate 10, range 20, 360 samples,
16 layers, a 1.0 rad vertical FOV, a full circle (as the literal
6.283185307179586 in one and ${2*pi} in the other) and GPU acceleration.
Both now read xacro properties defined in sensor.xacro, so a changed
default cannot leave one path on the old scan.

Rendering is byte-identical before and after with Noetic xacro 1.14.20
for: the SDF wrapper with no arguments; with only namespace and pose;
with every override as the FS150 renderer passes them (cpu, 20 Hz, 8 m,
720x32, pi/pi); the macro included from a URDF with only namespace and
pose; and with every parameter as the Mecanum model passes them.

Ported from the earlier local branch perf/gazebo-100-robots (de63856),
extended to horizontal_fov and acceleration, which were added since.
The FS150, Scout and Mecanum launch files and Core still pass every scan
parameter explicitly, so this does not change any Experiment's sensor.

File: xgc2_simple_lidar/models/sensor.sdf.xacro (robot description, xacro)
@@ -4,11 +4,12 @@
   <xacro:arg name="namespace" default="/robot"/>
   <xacro:arg name="pose" default="0 0 0 0 0 0"/>
-  <xacro:arg name="rate" default="10"/>
-  <xacro:arg name="max_range" default="20"/>
-  <xacro:arg name="samples" default="360"/>
-  <xacro:arg name="layers" default="16"/>
-  <xacro:arg name="vertical_fov" default="1.0"/>
-  <xacro:arg name="horizontal_fov" default="6.283185307179586"/>
-  <xacro:arg name="acceleration" default="gpu"/>
+  <!-- Optional overrides; their defaults are the macro's, from sensor.xacro. -->
+  <xacro:arg name="rate" default="${str(xgc2_simple_lidar_default_rate)}"/>
+  <xacro:arg name="max_range" default="${str(xgc2_simple_lidar_default_max_range)}"/>
+  <xacro:arg name="samples" default="${str(xgc2_simple_lidar_default_samples)}"/>
+  <xacro:arg name="layers" default="${str(xgc2_simple_lidar_default_layers)}"/>
+  <xacro:arg name="vertical_fov" default="${str(xgc2_simple_lidar_default_vertical_fov)}"/>
+  <xacro:arg name="horizontal_fov" default="${str(xgc2_simple_lidar_default_horizontal_fov)}"/>
+  <xacro:arg name="acceleration" default="${str(xgc2_simple_lidar_default_acceleration)}"/>
   <xacro:xgc2_simple_lidar_sensor namespace="$(arg namespace)" pose="$(arg pose)"
     rate="$(arg rate)" max_range="$(arg max_range)" samples="$(arg samples)"

File: xgc2_simple_lidar/models/sensor.xacro (robot description, xacro)
@@ -1,5 +1,14 @@
 <?xml version="1.0"?>
 <robot xmlns:xacro="http://www.ros.org/wiki/xacro">
-  <xacro:macro name="xgc2_simple_lidar_sensor" params="namespace pose rate:=10 max_range:=20 samples:=360 layers:=16 vertical_fov:=1.0 horizontal_fov:=${2*pi} acceleration:=gpu">
+  <!-- The only definition of the scan defaults. The macro parameters and the
+       sensor.sdf.xacro arguments both read these properties. -->
+  <xacro:property name="xgc2_simple_lidar_default_rate" value="10"/>
+  <xacro:property name="xgc2_simple_lidar_default_max_range" value="20"/>
+  <xacro:property name="xgc2_simple_lidar_default_samples" value="360"/>
+  <xacro:property name="xgc2_simple_lidar_default_layers" value="16"/>
+  <xacro:property name="xgc2_simple_lidar_default_vertical_fov" value="1.0"/>
+  <xacro:property name="xgc2_simple_lidar_default_horizontal_fov" value="${2*pi}"/>
+  <xacro:property name="xgc2_simple_lidar_default_acceleration" value="gpu"/>
+  <xacro:macro name="xgc2_simple_lidar_sensor" params="namespace pose rate:=${xgc2_simple_lidar_default_rate} max_range:=${xgc2_simple_lidar_default_max_range} samples:=${xgc2_simple_lidar_default_samples} layers:=${xgc2_simple_lidar_default_layers} vertical_fov:=${xgc2_simple_lidar_default_vertical_fov} horizontal_fov:=${xgc2_simple_lidar_default_horizontal_fov} acceleration:=${xgc2_simple_lidar_default_acceleration}">
     <sensor name="simple_lidar" type="${dict(cpu='ray', gpu='gpu_ray')[acceleration]}">
       <pose>${pose}</pose>
